Commit message: the vibraitons are the problem

File: mur_description/urdf/mur_base.xacro (robot description, xacro)
@@ -2,5 +2,5 @@
 <robot xmlns:xacro="http://www.ros.org/wiki/xacro">
     <!-- Import macro files -->
-    <xacro:include filename="$(find uuv_descriptions)/models/common/urdf/common.urdf.xacro" />
+    <xacro:include filename="$(find uuv_descriptions)/urdf/common.urdf.xacro" />
     <xacro:include filename="$(find uuv_sensor_ros_plugins)/urdf/sensor_snippets.xacro"/>
     <xacro:include filename="$(find uuv_gazebo_ros_plugins)/urdf/snippets.xacro"/>
@@ -12,5 +12,5 @@
     <xacro:property name="rho" value="1027.0"/>
     <xacro:property name="visual_mesh_file" value="file://$(find mur_description)/mesh/mur.dae"/>
-    <xacro:property name="collision_mesh_file" value="file://$(find mur_description)/mesh/mur.stl"/>
+    <xacro:property name="collision_mesh_file" value="file://$(find mur_description)/mesh/mur.dae"/>
     <xacro:property name="prop_mesh_file" value="file://$(find mur_description)/mesh/mur_prop.dae"/>
     <xacro:macro name="mur_base" params="namespace debug">

File: mur_description/urdf/mur_sensors.xacro (robot description, xacro)
@@ -12,7 +12,7 @@
     </xacro:default_pressure>
     <!-- IMU  -->
-    <xacro:default_imu namespace="${namespace}" parent_link="${namespace}/base_link">
+    <xacro:default_imu_enu namespace="${namespace}" parent_link="${namespace}/base_link">
       <origin xyz="0 0 0" rpy="0 0 0"/>
-    </xacro:default_imu>
+    </xacro:default_imu_enu>
     <!-- Mount a camera -->
     <xacro:regular_camera_plugin_macro

Commit message: New drag coefficients

File: mur_description/urdf/mur_base.xacro (robot description, xacro)
@@ -7,6 +7,6 @@
     <!--xacro:include filename="$(find mur_description)/urdf/mur_snippets.xacro"/-->
     <!-- Properties -->
-    <xacro:property name="mass" value="8.37"/>
-    <xacro:property name="volume" value="0.004837965"/>
+    <xacro:property name="mass" value="8.96"/>
+    <xacro:property name="volume" value="0.008550699"/>
     <xacro:property name="cob" value="0 0 0"/>
     <xacro:property name="rho" value="1027.0"/>
@@ -68,5 +68,5 @@
               </linear_damping-->
               <quadratic_damping>
-                -26.5547 -17.1505 -37.8527 -0.00711 -0.0123 -0.45725
+                -17.4666 -50.8618 -55.7484 -0.00711 -0.0123 -0.45725
               </quadratic_damping>
             </hydrodynamic_model>

Commit message: Check PID

File: mur_description/urdf/mur_base.xacro (robot description, xacro)
@@ -7,5 +7,5 @@
     <!--xacro:include filename="$(find mur_description)/urdf/mur_snippets.xacro"/-->
     <!-- Properties -->
-    <xacro:property name="mass" value="8.96"/>
+    <xacro:property name="mass" value="9.6"/> <!--The real value is 8.6, but it was changed for the simulation. The real life add 1kg to the robot.-->
     <xacro:property name="volume" value="0.008550699"/>
     <xacro:property name="cob" value="0 0 0"/>

Commit message: Added latest changes to simulation

File: mur_description/urdf/mur_base.xacro (robot description, xacro)
@@ -31,7 +31,7 @@
               <mass value="${mass}" />
               <origin xyz="0 0 0" rpy="0 0 0"/>
-              <inertia ixx="0.38467478" ixy="0" ixz="0"
-                       iyy="0.16784643" iyz="0"
-                       izz="0.46539770" />
+              <inertia ixx="0.2222" ixy="0" ixz="0"
+                       iyy="0.1496" iyz="0"
+                       izz="0.320" />
             </inertial>
         </link>
@@ -49,10 +49,10 @@
               <type>fossen</type>
               <added_mass>
-                8.37    0       0       0       0       0
-                0       8.37    0       0       0       0
-                0       0       8.37    0       0       0
-                0       0       0       0.384   0       0
-                0       0       0       0       0.465   0
-                0       0       0       0       0       0.167
+                9.6     0       0       0       0       0
+                0       9.60    0       0       0       0
+                0       0       9.60    0       0       0
+                0       0       0       1       0       0
+                0       0       0       0       1       0
+                0       0       0       0       0       1
               </added_mass>
               <!--<linear_damping_forward_speed>
@@ -68,5 +68,5 @@
               </linear_damping-->
               <quadratic_damping>
-                -17.4666 -50.8618 -55.7484 -0.00711 -0.0123 -0.45725
+                -17.4666 -50.8618 -55.7484 -0.47 -0.34 -0.99
               </quadratic_damping>
             </hydrodynamic_model>

File: mur_description/urdf/mur_base_ident.xacro (robot description, xacro)
@@ -32,7 +32,7 @@
               <mass value="${mass}" />
               <origin xyz="0 0 0" rpy="0 0 0"/>
-              <inertia ixx="0.38467478" ixy="0" ixz="0"
-                       iyy="0.16784643" iyz="0"
-                       izz="0.46539770" />
+              <inertia ixx="0.22228451" ixy="0" ixz="0"
+                       iyy="0.14925489" iyz="0"
+                       izz="0.32042275" />
             </inertial>
         </link>
@@ -86,5 +86,5 @@
             <origin xyz="0 0 0" rpy="0 0 0" />
             <geometry>
-              <box size="2.5 4.5 0.01" />
+              <box size="4.5 2.5 0.01" />
             </geometry>
             <material name="grey">
@@ -95,5 +95,5 @@
             <origin xyz="0 0 0" rpy="0 0 0" />
             <geometry>
-              <box size="2.5 4.5 0.01" />
+              <box size="4.5 2.5 0.01" />
             </geometry>
             <surface>
@@ -109,7 +109,7 @@
             <mass value="50" />
             <origin xyz="0.0 0.0 0.0"/>
-            <inertia ixx="0.0" ixy="0.0" ixz="0.0"
-              iyy="0.0" iyz="0.0"
-              izz="0.0" />
+            <inertia ixx="10.0" ixy="0.0" ixz="0.0"
+              iyy="10.0" iyz="0.0"
+              izz="10.0" />
           </inertial>
         </link>
