Commit message: EKF working with one aruco

File: mur_description/urdf/mur_sensors.xacro (robot description, xacro)
@@ -3,15 +3,39 @@
     <!-- Mount a 3D pose sensor -->
     <xacro:default_pose_3d namespace="${namespace}" parent_link="${namespace}/base_link" />
-    <!-- Side scan sonar -->
-    <xacro:sidescan_sonar namespace="${namespace}" parent_link="${namespace}/base_link" suffix="main">
-      <origin xyz="0.41225 0.1498 -0.04615" rpy="${0.5*pi} ${-5*d2r+pi/3.0} ${0.5*pi}" />
-    </xacro:sidescan_sonar>
+    <!-- Sonar -->
+    <!-- Inspired by https://www.tritech.co.uk/product/small-rov-mechanical-sector-scanning-sonar-tritech-micron-->
+    <xacro:macro name="micron_sonar_tritech" params="namespace parent_link *origin">
+      <xacro:multibeam_sonar
+        namespace="${namespace}"
+        suffix=""
+        parent_link="${parent_link}"
+        topic="sonar"
+        mass="0.015"
+        update_rate="10"
+        samples="250"
+        fov="3.92"
+        range_min="0.3"
+        range_max="75.0"
+        range_stddev="0.0075"
+        mesh="">
+        <inertia ixx="0.00001" ixy="0.0" ixz="0.0" iyy="0.00001" iyz="0.0" izz="0.00001" />
+        <xacro:insert_block name="origin" />
+        <visual>
+          <geometry>
+            <mesh filename="file://$(find mur_description)/mesh/Micron DST Sonar.dae" scale="1 1 1"/>
+          </geometry>
+        </visual>
+      </xacro:multibeam_sonar>
+    </xacro:macro>
+    <xacro:micron_sonar_tritech namespace="${namespace}" parent_link="${namespace}/base_link">
+      <origin xyz="0 0.21 0.057" rpy="0 0 ${0.5*pi}" />
+    </xacro:micron_sonar_tritech>
     <!-- Pressure -->
     <xacro:default_pressure namespace="${namespace}" parent_link="${namespace}/base_link">
-      <origin xyz="0 0 0" rpy="0 0 0"/>
+      <origin xyz="-0.055 -0.160 0" rpy="${0.5*pi} 0 0"/>
     </xacro:default_pressure>
     <!-- IMU  -->
     <xacro:default_imu_enu namespace="${namespace}" parent_link="${namespace}/base_link">
-      <origin xyz="0 0 0" rpy="0 0 0"/>
+      <origin xyz="-0.055 -0.08 0" rpy="0 0 0"/>
     </xacro:default_imu_enu>
     <!-- Mount a camera -->
@@ -23,11 +47,11 @@
         mass="0.1"
         update_rate="30"
-        hfov="1.5125"
-        width="768"
-        height="492"
-        stddev="0.02"
+        hfov="0.75"
+        width="640"
+        height="480"
+        stddev="0.005"
         scale="1.0">
         <inertia ixx="0.00001" ixy="0.0" ixz="0.0" iyy="0.00001" iyz="0.0" izz="0.00001" />
-        <origin xyz="0.055 0.160 0" rpy="0 0 ${0.5*pi}"/>
+        <origin xyz="-0.055 0.160 0" rpy="0 0 ${0.5*pi}"/>
     </xacro:regular_camera_plugin_macro>
     <!-- Mount a GPS.

Commit message: Supervisor was added

File: mur_description/urdf/mur_sensors.xacro (robot description, xacro)
@@ -39,11 +39,27 @@
       <origin xyz="-0.055 -0.08 0" rpy="0 0 0"/>
     </xacro:default_imu_enu>
-    <!-- Mount a camera -->
+    <!-- Mount a camera # 1-->
     <xacro:regular_camera_plugin_macro
         namespace="${namespace}"
-        suffix=""
+        suffix="1"
         parent_link="${namespace}/base_link"
         topic="camera"
-        mass="0.1"
+        mass="0.075"
+        update_rate="30"
+        hfov="0.75"
+        width="1280"
+        height="720"
+        stddev="0.005"
+        scale="1.0">
+        <inertia ixx="0.00001" ixy="0.0" ixz="0.0" iyy="0.00001" iyz="0.0" izz="0.00001" />
+        <origin xyz="-0.055 0.160 0" rpy="0 0 ${0.5*pi}"/>
+    </xacro:regular_camera_plugin_macro>
+    <!-- Mount a camera # 2-->
+    <xacro:regular_camera_plugin_macro
+        namespace="${namespace}"
+        suffix="2"
+        parent_link="${namespace}/base_link"
+        topic="camera"
+        mass="0.05"
         update_rate="30"
         hfov="0.75"
@@ -53,5 +69,5 @@
         scale="1.0">
         <inertia ixx="0.00001" ixy="0.0" ixz="0.0" iyy="0.00001" iyz="0.0" izz="0.00001" />
-        <origin xyz="-0.055 0.160 0" rpy="0 0 ${0.5*pi}"/>
+        <origin xyz="-0.055 0 -0.06" rpy="0 ${0.5*pi} ${0.5*pi}"/>
     </xacro:regular_camera_plugin_macro>
     <!-- Mount a GPS.
