Commit message: Run just rviz and gazebo in backend

File: mur_description/urdf/mur_base_5.xacro (robot description, xacro)
@@ -7,5 +7,5 @@
     <!--xacro:include filename="$(find mur_description)/urdf/mur_snippets.xacro"/-->
     <!-- Properties -->
-    <xacro:property name="mass" value="9.6"/> <!--The real value is 8.6, but it was changed for the simulation. The real life add 1kg to the robot.-->
+    <xacro:property name="mass" value="10.6"/> <!--The real value is 8.6, but it was changed for the simulation. The real life add 1kg to the robot.-->
     <xacro:property name="volume" value="0.008550699"/>
     <xacro:property name="cob" value="0 0 0"/>
@@ -49,10 +49,10 @@
               <type>fossen</type>
               <added_mass>
-                9.6     0       0       0       0       0
-                0       9.60    0       0       0       0
-                0       0       9.60    0       0       0
-                0       0       0       1       0       0
-                0       0       0       0       1       0
-                0       0       0       0       0       1
+                2.13     0       0       0       0       0
+                0       8.0257    0       0       0       0
+                0       0       7.3667    0       0       0
+                0       0       0       0.2222       0       0
+                0       0       0       0       0.1492       0
+                0       0       0       0       0       0.3209
               </added_mass>
               <!--<linear_damping_forward_speed>
@@ -65,8 +65,8 @@
               </linear_damping_forward_speed>-->
               <!--linear_damping>
-                -1.1033 -2.2187 -0.03113 -0.1 -0.1 -0.1
+                -0 -0 -0 -15.3427 -44.6770 -48.9694
               </linear_damping-->
               <quadratic_damping>
-                -17.4666 -50.8618 -55.7484 -0.47 -0.34 -0.99
+                -17.4666 -50.8618 -55.7484 -84.5403 -50.6692 -77.13
               </quadratic_damping>
             </hydrodynamic_model>

File: mur_description/urdf/mur_base_ident.xacro (robot description, xacro)
@@ -7,10 +7,10 @@
     <!--xacro:include filename="$(find mur_description)/urdf/mur_snippets.xacro"/-->
     <!-- Properties -->
-    <xacro:property name="mass" value="9.6"/> <!--The real value is 8.6, but it was changed for the simulation. The real life add 1kg to the robot.-->
+    <xacro:property name="mass" value="10.6"/> <!--The real value is 8.6, but it was changed for the simulation. The real life add 1kg to the robot.-->
     <xacro:property name="volume" value="0.008550699"/>
     <xacro:property name="cob" value="0 0 0"/>
     <xacro:property name="rho" value="1027.0"/>
-    <xacro:property name="visual_mesh_file" value="file://$(find mur_description)/mesh/mur.dae"/>
-    <xacro:property name="collision_mesh_file" value="file://$(find mur_description)/mesh/mur.dae"/>
+    <xacro:property name="visual_mesh_file" value="file://$(find mur_description)/mesh/mur_5.dae"/>
+    <xacro:property name="collision_mesh_file" value="file://$(find mur_description)/mesh/mur_5.dae"/>
     <xacro:property name="prop_mesh_file" value="file://$(find mur_description)/mesh/mur_prop.dae"/>
     <xacro:macro name="mur_base_ident" params="namespace debug">
@@ -38,10 +38,10 @@
         </link>
 <!-- JOINT BETWEEN ROBOT AND ARM -->
-        <joint name="mur_arm_joint" type="continuous">
+        <joint name="mur_arm_joint" type="revolute">
           <parent link="${namespace}/base_link"/>
           <child link="${namespace}/arm_base_link" />
           <origin xyz="0 0 0" rpy="0 0 0"/>
           <axis xyz="1 1 0"/>
-          <limit effort="9999999999999" velocity="999999999999"/>
+          <limit effort="9999999999999" velocity="999999999999" lower="-0.35" upper="0.35"/>
         </joint>
 <!-- ARM -->
@@ -127,10 +127,10 @@
               <type>fossen</type>
               <added_mass>
-                8.37    0       0       0       0       0
-                0       8.37    0       0       0       0
-                0       0       8.37    0       0       0
-                0       0       0       0.384   0       0
-                0       0       0       0       0.465   0
-                0       0       0       0       0       0.167
+                2.13     0       0       0       0       0
+                0       8.0257    0       0       0       0
+                0       0       7.3667    0       0       0
+                0       0       0       0.2222       0       0
+                0       0       0       0       0.1492       0
+                0       0       0       0       0       0.3209
               </added_mass>
               <!--<linear_damping_forward_speed>
@@ -146,5 +146,5 @@
               </linear_damping-->
               <quadratic_damping>
-                -17.4666 -50.8618 -55.7484 -0.00711 -0.0123 -0.45725
+                -17.4666 -50.8618 -55.7484 -0.47 -0.34 -0.99
               </quadratic_damping>
             </hydrodynamic_model>
@@ -191,5 +191,5 @@
       </gazebo>
       <xacro:include filename="$(find mur_description)/urdf/mur_sensors.xacro"/>
-      <xacro:include filename="$(find mur_description)/urdf/mur_actuators.xacro"/>
+      <xacro:include filename="$(find mur_description)/urdf/mur_actuators_5.xacro"/>
     </xacro:macro>
 </robot>

Commit message: model was edited for VSC

File: mur_description/urdf/mur_base_5.xacro (robot description, xacro)
@@ -64,9 +64,9 @@
                 0       -34     0       0       0       -32
               </linear_damping_forward_speed>-->
-              <!--linear_damping>
-                -0 -0 -0 -15.3427 -44.6770 -48.9694
-              </linear_damping-->
+              <linear_damping>
+                -0 -0 -0 -0.6508 -1.0745 -0.3834
+              </linear_damping>
               <quadratic_damping>
-                -17.4666 -50.8618 -55.7484 -84.5403 -50.6692 -77.13
+                -17.4666 -50.8618 -55.7484 -15.2562 -11.2216 -32.0758
               </quadratic_damping>
             </hydrodynamic_model>

File: mur_description/urdf/mur_base_ident.xacro (robot description, xacro)
@@ -40,8 +40,42 @@
         <joint name="mur_arm_joint" type="revolute">
           <parent link="${namespace}/base_link"/>
-          <child link="${namespace}/arm_base_link" />
+          <child link="${namespace}/arm0_base_link" />
           <origin xyz="0 0 0" rpy="0 0 0"/>
           <axis xyz="1 1 0"/>
           <limit effort="9999999999999" velocity="999999999999" lower="-0.35" upper="0.35"/>
+        </joint>
+        <link name="${namespace}/arm0_base_link">
+          <visual>
+            <origin xyz="0 0 0.05" rpy="0 0 0" />
+            <geometry>
+                <cylinder length="0.1" radius="0.005"/>
+                <!--box size="2 4.3 0.01" /-->
+            </geometry>
+            <material name="red">
+              <color rgba="1 0 0 1"/>
+            </material>
+          </visual>
+          <collision>
+            <origin xyz="0 0 0" rpy="0 0 0" />
+            <geometry>
+            <cylinder length="0.6" radius="0.2"/>
+            <!--cylinder length="1.5" radius="0.005"/-->
+            <!--box size="2 4.3 0.01" /-->
+            </geometry>
+          </collision>
+          <inertial>
+            <mass value="0.001" />
+            <origin xyz="0.0 0.0 0.0"/>
+            <inertia ixx="0.0" ixy="0.0" ixz="0.0"
+              iyy="0.0" iyz="0.0"
+              izz="0.0" />
+          </inertial>
+        </link>
+        <joint name="mur_arm0_joint" type="prismatic">
+          <parent link="${namespace}/arm0_base_link"/>
+          <child link="${namespace}/arm_base_link" />
+          <origin xyz="0 0 0" rpy="0 0 0"/>
+          <axis xyz="0 0 1"/>
+          <limit effort="9999999999999" velocity="999999999999" lower="-0.15" upper="0.15"/>
         </joint>
 <!-- ARM -->
@@ -107,9 +141,9 @@
           </collision>
           <inertial>
-            <mass value="50" />
+            <mass value="500" />
             <origin xyz="0.0 0.0 0.0"/>
-            <inertia ixx="10.0" ixy="0.0" ixz="0.0"
-              iyy="10.0" iyz="0.0"
-              izz="10.0" />
+            <inertia ixx="100.0" ixy="0.0" ixz="0.0"
+              iyy="100.0" iyz="0.0"
+              izz="100.0" />
           </inertial>
         </link>

File: mur_description/urdf/mur_sensors.xacro (robot description, xacro)
@@ -11,5 +11,5 @@
         parent_link="${parent_link}"
         topic="sonar"
-        mass="0.015"
+        mass="0.180"
         update_rate="10"
         samples="250"

Commit message: Smooth motors behaviour has been added
It doesnt work so good

File: mur_description/urdf/mur_base_5.xacro (robot description, xacro)
@@ -65,8 +65,8 @@
               </linear_damping_forward_speed>-->
               <linear_damping>
-                -0 -0 -0 -0.6508 -1.0745 -0.3834
+                -0 -0 -0 -0.4721 -0.3472 -0.9926
               </linear_damping>
               <quadratic_damping>
-                -17.4666 -50.8618 -55.7484 -15.2562 -11.2216 -32.0758
+                -17.4666 -50.8618 -55.7484 -1.6901 -1.0130 -3.5534
               </quadratic_damping>
             </hydrodynamic_model>

File: mur_description/urdf/mur_base_ident.xacro (robot description, xacro)
@@ -42,5 +42,5 @@
           <child link="${namespace}/arm0_base_link" />
           <origin xyz="0 0 0" rpy="0 0 0"/>
-          <axis xyz="1 1 1"/>
+          <axis xyz="1 0 0"/>
           <limit effort="9999999999999" velocity="999999999999" lower="-0.35" upper="0.35"/>
         </joint>

Commit message: Floats were added in URDF

File: mur_description/urdf/mur_base_5.xacro (robot description, xacro)
@@ -7,7 +7,7 @@
     <!--xacro:include filename="$(find mur_description)/urdf/mur_snippets.xacro"/-->
     <!-- Properties -->
-    <xacro:property name="mass" value="10.6"/> <!--The real value is 8.6, but it was changed for the simulation. The real life add 1kg to the robot.-->
-    <xacro:property name="volume" value="0.008550699"/>
-    <xacro:property name="cob" value="0 0 0"/>
+    <xacro:property name="mass" value="9.7"/> <!--The real value is 8.6, but it was changed for the simulation. The real life add 1kg to the robot.-->
+    <xacro:property name="volume" value="0.010050699"/>
+    <xacro:property name="cob" value="0 0.008 0.03"/>
     <xacro:property name="rho" value="1027.0"/>
     <xacro:property name="visual_mesh_file" value="file://$(find mur_description)/mesh/mur_5.dae"/>

Commit message: Expor videos launch has been added

File: mur_description/urdf/mur_base_5.xacro (robot description, xacro)
@@ -8,5 +8,5 @@
     <!-- Properties -->
     <xacro:property name="mass" value="9.7"/> <!--The real value is 8.6, but it was changed for the simulation. The real life add 1kg to the robot.-->
-    <xacro:property name="volume" value="0.010050699"/>
+    <xacro:property name="volume" value="0.0112"/>
     <xacro:property name="cob" value="0 0.008 0.03"/>
     <xacro:property name="rho" value="1027.0"/>
