Commit message: Updated to melodic

File: mur_description/urdf/mur_actuators_5.xacro (robot description, xacro)
@@ -28,14 +28,14 @@
     </xacro:macro>
     <xacro:thruster_macro namespace="${namespace}" thruster_id="0">
-        <origin xyz="0.197 0.18022 0.074" rpy="0 ${-95*pi/180} ${-pi/2}" />
+        <origin xyz="0.2 0.1742 0.0745" rpy="0 ${-85*pi/180} ${-pi/2}" />
+    </xacro:thruster_macro>
+    <xacro:thruster_macro namespace="${namespace}" thruster_id="1">
+        <origin xyz="0.2 -0.1742 0.0745" rpy="0 ${-95*pi/180} ${-pi/2}" />
     </xacro:thruster_macro>
     <xacro:thruster_macro namespace="${namespace}" thruster_id="2">
-        <origin xyz="-0.197 -0.18022 0.074" rpy="0 ${-85*pi/180} ${-pi/2}" />
-    </xacro:thruster_macro>
-    <xacro:thruster_macro namespace="${namespace}" thruster_id="1">
-        <origin xyz="0.197 -0.18022 0.074" rpy="0 ${-85*pi/180} ${-pi/2}" />
+        <origin xyz="-0.2 -0.1742 0.0745" rpy="0 ${-95*pi/180} ${-pi/2}" />
     </xacro:thruster_macro>
     <xacro:thruster_macro namespace="${namespace}" thruster_id="3">
-        <origin xyz="-0.197 0.18022 0.074" rpy="0 ${-95*pi/180} ${-pi/2}" />
+        <origin xyz="-0.2 0.1742 0.0745" rpy="0 ${-85*pi/180} ${-pi/2}" />
     </xacro:thruster_macro>
 </robot>

Commit message: New roslaunch for real robot

File: mur_description/urdf/mur_actuators_5.xacro (robot description, xacro)
@@ -28,14 +28,14 @@
     </xacro:macro>
     <xacro:thruster_macro namespace="${namespace}" thruster_id="0">
-        <origin xyz="0.2 0.1742 0.0745" rpy="0 ${-85*pi/180} ${-pi/2}" />
+        <origin xyz="0.2 0.1742 0.0745" rpy="0 ${-80*pi/180} ${-pi/2}" />
     </xacro:thruster_macro>
     <xacro:thruster_macro namespace="${namespace}" thruster_id="1">
-        <origin xyz="0.2 -0.1742 0.0745" rpy="0 ${-95*pi/180} ${-pi/2}" />
+        <origin xyz="0.2 -0.1742 0.0745" rpy="0 ${-100*pi/180} ${-pi/2}" />
     </xacro:thruster_macro>
     <xacro:thruster_macro namespace="${namespace}" thruster_id="2">
-        <origin xyz="-0.2 -0.1742 0.0745" rpy="0 ${-95*pi/180} ${-pi/2}" />
+        <origin xyz="-0.2 -0.1742 0.0745" rpy="0 ${-100*pi/180} ${-pi/2}" />
     </xacro:thruster_macro>
     <xacro:thruster_macro namespace="${namespace}" thruster_id="3">
-        <origin xyz="-0.2 0.1742 0.0745" rpy="0 ${-85*pi/180} ${-pi/2}" />
+        <origin xyz="-0.2 0.1742 0.0745" rpy="0 ${-80*pi/180} ${-pi/2}" />
     </xacro:thruster_macro>
 </robot>

File: mur_description/urdf/mur_base_ident.xacro (robot description, xacro)
@@ -42,5 +42,5 @@
           <child link="${namespace}/arm0_base_link" />
           <origin xyz="0 0 0" rpy="0 0 0"/>
-          <axis xyz="1 1 0"/>
+          <axis xyz="1 1 1"/>
           <limit effort="9999999999999" velocity="999999999999" lower="-0.35" upper="0.35"/>
         </joint>

File: mur_description/urdf/mur_sensors.xacro (robot description, xacro)
@@ -13,5 +13,5 @@
         mass="0.180"
         update_rate="10"
-        samples="250"
+        samples="50"
         fov="3.92"
         range_min="0.3"

Commit message: Bouyancy has been corrected

File: mur_description/urdf/mur_actuators_5.xacro (robot description, xacro)
@@ -21,21 +21,21 @@
         </dynamics>
         <xacro:thruster_cf_dead_zone_macro
-          rotor_constant_l="0.096047"
-          rotor_constant_r="0.111192"
-          delta_l="-3.5604"
-          delta_r="2.5132"/>
+          rotor_constant_l="0.000275"
+          rotor_constant_r="0.000275"
+          delta_l="0"
+          delta_r="0"/>
       </xacro:generic_thruster_macro>
     </xacro:macro>
     <xacro:thruster_macro namespace="${namespace}" thruster_id="0">
-        <origin xyz="0.2 0.1742 0.0745" rpy="0 ${-80*pi/180} ${-pi/2}" />
+        <origin xyz="0.2 0.1742 0.0745" rpy="0 ${-95*pi/180} ${-pi/2}" />
     </xacro:thruster_macro>
     <xacro:thruster_macro namespace="${namespace}" thruster_id="1">
-        <origin xyz="0.2 -0.1742 0.0745" rpy="0 ${-100*pi/180} ${-pi/2}" />
+        <origin xyz="0.2 -0.1742 0.0745" rpy="0 ${-85*pi/180} ${-pi/2}" />
     </xacro:thruster_macro>
     <xacro:thruster_macro namespace="${namespace}" thruster_id="2">
-        <origin xyz="-0.2 -0.1742 0.0745" rpy="0 ${-100*pi/180} ${-pi/2}" />
+        <origin xyz="-0.2 -0.1742 0.0745" rpy="0 ${-85*pi/180} ${-pi/2}" />
     </xacro:thruster_macro>
     <xacro:thruster_macro namespace="${namespace}" thruster_id="3">
-        <origin xyz="-0.2 0.1742 0.0745" rpy="0 ${-80*pi/180} ${-pi/2}" />
+        <origin xyz="-0.2 0.1742 0.0745" rpy="0 ${-95*pi/180} ${-pi/2}" />
     </xacro:thruster_macro>
 </robot>

File: mur_description/urdf/mur_base_5.xacro (robot description, xacro)
@@ -7,11 +7,10 @@
     <!--xacro:include filename="$(find mur_description)/urdf/mur_snippets.xacro"/-->
     <!-- Properties -->
-    <xacro:property name="mass" value="9.7"/> <!--The real value is 8.6, but it was changed for the simulation. The real life add 1kg to the robot.-->
-    <xacro:property name="volume" value="0.0112"/>
-    <xacro:property name="cob" value="0 0.008 0.03"/>
-    <xacro:property name="rho" value="1027.0"/>
+    <xacro:property name="mass" value="11.4"/> <!--The real value is 11.4, but it was changed for the simulation. The real life add 1kg to the robot.-->
+    <xacro:property name="volume" value="0.012349"/> <!--0.012349-->
+    <xacro:property name="cob" value="0 0.005 0.075"/>
+    <xacro:property name="rho" value="1000.0"/>
     <xacro:property name="visual_mesh_file" value="file://$(find mur_description)/mesh/mur_5.dae"/>
     <xacro:property name="collision_mesh_file" value="file://$(find mur_description)/mesh/mur_5.dae"/>
-    <xacro:property name="prop_mesh_file" value="file://$(find mur_description)/mesh/mur_prop.dae"/>
     <xacro:macro name="mur_base_5" params="namespace debug">
         <link name="${namespace}/base_link">
@@ -49,9 +48,9 @@
               <type>fossen</type>
               <added_mass>
-                2.13     0       0       0       0       0
-                0       8.0257    0       0       0       0
-                0       0       7.3667    0       0       0
-                0       0       0       0.2222       0       0
-                0       0       0       0       0.1492       0
+                ${mass*0.2404}  0       0       0       0       0
+                0       ${mass*0.9024}  0       0       0       0
+                0       0       ${mass*0.8283}  0       0       0
+                0       0       0       0.2222  0       0
+                0       0       0       0       0.1492  0
                 0       0       0       0       0       0.3209
               </added_mass>
@@ -65,8 +64,8 @@
               </linear_damping_forward_speed>-->
               <linear_damping>
-                -0 -0 -0 -0.4721 -0.3472 -0.9926
+                -0.6508 -1.0745 -0.3834 -5.1103 -3.7588 -14.3219
               </linear_damping>
               <quadratic_damping>
-                -17.4666 -50.8618 -55.7484 -1.6901 -1.0130 -3.5534
+                -17.4666 -50.8618 -55.7484 -743.0698 -546.5597 -677.9363
               </quadratic_damping>
             </hydrodynamic_model>
