Commit message: SIm with right thruster model

File: mur_description/urdf/mur_actuators.xacro (robot description, xacro)
@@ -11,12 +11,19 @@
     <xacro:macro name="thruster_macro"
       params="namespace thruster_id *origin">
-      <xacro:thruster_module_first_order_basic_fcn_macro
+      <xacro:generic_thruster_macro
         namespace="${namespace}"
         thruster_id="${thruster_id}"
-        mesh_filename="${prop_mesh_file}"
-        dyn_time_constant="0.05"
-        rotor_constant="0.00031">
+        mesh_filename="${prop_mesh_file}">
         <xacro:insert_block name="origin"/>
-      </xacro:thruster_module_first_order_basic_fcn_macro>
+        <dynamics>
+          <type>FirstOrder</type>
+          <timeConstant>0.52</timeConstant>
+        </dynamics>
+        <xacro:thruster_cf_dead_zone_macro
+          rotor_constant_l="0.096047"
+          rotor_constant_r="0.111192"
+          delta_l="-3.5604"
+          delta_r="2.5132"/>
+      </xacro:generic_thruster_macro>
     </xacro:macro>
     <xacro:thruster_macro namespace="${namespace}" thruster_id="0">

File: mur_description/urdf/mur_base.xacro (robot description, xacro)
@@ -4,6 +4,6 @@
     <xacro:include filename="$(find uuv_descriptions)/models/common/urdf/common.urdf.xacro" />
     <xacro:include filename="$(find uuv_sensor_ros_plugins)/urdf/sensor_snippets.xacro"/>
-    <xacro:include filename="$(find mur_description)/urdf/mur_snippets.xacro"/>
     <xacro:include filename="$(find uuv_gazebo_ros_plugins)/urdf/snippets.xacro"/>
+    <!--xacro:include filename="$(find mur_description)/urdf/mur_snippets.xacro"/-->
     <!-- Properties -->
     <xacro:property name="mass" value="8.37"/>

File: mur_description/urdf/mur_snippets.xacro (robot description, xacro)
@@ -7,10 +7,10 @@
   over propeller's frame X-axis in DAE (Collada) or STL format.
   -->
-  <xacro:property name="prop_mesh_file" value="file://$(find mur_description)/meshes/mur_prop.dae"/>
+  <xacro:property name="prop_mesh_file" value="file://$(find mur_description)/mesh/mur_prop.dae"/>
   <!--
     Thruster macro with integration of joint and link. The thrusters should
     be initialized in the actuators.xacro file.
   -->
-  <xacro:macro name="thruster_macro" params="robot_namespace thruster_id *origin">
+  <xacro:macro name="thruster_macro" params="namespace thruster_id *origin">
     <!--
     Dummy link as place holder for the thruster frame,
@@ -18,5 +18,5 @@
     of the vehicle and may cause internal collisions if set otherwise
     -->
-    <link name="${robot_namespace}/thruster_${thruster_id}">
+    <link name="${namespace}/thruster_${thruster_id}">
       <visual>
         <geometry>
@@ -33,17 +33,17 @@
     </link>
     <!-- Joint between thruster link and vehicle base link -->
-    <joint name="${robot_namespace}/thruster_${thruster_id}_joint" type="continuous">
+    <joint name="${namespace}/thruster_${thruster_id}_joint" type="continuous">
       <xacro:insert_block name="origin" />
       <axis xyz="1 0 0" />
-      <parent link="${robot_namespace}/base_link" />
-      <child link="${robot_namespace}/thruster_${thruster_id}" />
+      <parent link="${namespace}/base_link" />
+      <child link="${namespace}/thruster_${thruster_id}" />
     </joint>
     <gazebo>
       <!-- Thruster ROS plugin -->
-      <plugin name="${robot_namespace}_${thruster_id}_thruster_model" filename="libthruster_ros_plugin.so">
+      <plugin name="${namespace}_${thruster_id}_thruster_model" filename="libthruster_ros_plugin.so">
         <!-- Name of the thruster link -->
-        <linkName>${robot_namespace}/thruster_${thruster_id}</linkName>
+        <linkName>${namespace}/thruster_${thruster_id}</linkName>
         <!-- Name of the joint between thruster and vehicle base link -->
-        <jointName>${robot_namespace}/thruster_${thruster_id}_joint</jointName>
+        <jointName>${namespace}/thruster_${thruster_id}_joint</jointName>
         <!-- Make the thruster aware of its id -->
         <thrusterID>${thruster_id}</thrusterID>
@@ -55,6 +55,6 @@
         <clampMin>1100</clampMin>
         <!-- Minimum and maximum thrust force output allowed -->
-        <thrustMin>-30</thrustMin>
-        <thrustMax>34</thrustMax>
+        <thrustMin>-29.43</thrustMin>
+        <thrustMax>34.82</thrustMax>
         <!--
         Value from 0 to 1 to set the efficiency of the output thrust force
@@ -74,12 +74,12 @@
         which can be, e.g., the angular velocity of the propeller.
         -->
-        <!-- 1) Simple zero-order model -->
+        <!-- 1) Simple zero-order model
         <dynamics>
           <type>ZeroOrder</type>
-        </dynamics>
+        </dynamics>-->
         <!-- 2) First order model
         <dynamics>
           <type>FirstOrder</type>
-          <timeConstant>0.0</timeConstant>
+          <timeConstant>0.52</timeConstant>
         </dynamics>-->
         <!-- 3) Yoerger's nonlinear dynamic model
@@ -102,5 +102,5 @@
         <dynamics>
           <type>Bessa</type>
-          <Jmsp>0.0</Jmsp>
+          <Jmsp>0.0000091875</Jmsp>
           <Kv1>0.0</Kv1>
           <Kv2>0.0</Kv2>
@@ -129,8 +129,8 @@
         <conversion>
           <type>Bessa</type>
-          <rotorConstantL>0.0</rotorConstantL>
-          <rotorConstantR>0.0</rotorConstantR>
-          <deltaL>0.0</deltaL>
-          <deltaR>0.0</deltaR>
+          <rotorConstantL>0.0613125</rotorConstantL>
+          <rotorConstantR>0.09122</rotorConstantR>
+          <deltaL>1480</deltaL>
+          <deltaR>1520</deltaR>
         </conversion>-->
         <!-- 3) Linear interpolation
@@ -138,15 +138,15 @@
         you can enter samples of the curve's input and output values
         and the thruster output will be found through linear interpolation
-        of the given samples.-->
+        of the given samples.
         <conversion>
           <type>LinearInterp</type>
           <inputValues>0.0072  -10.6673</inputValues>
           <outputValues>0.0072  -10.6673</outputValues>
-        </conversion>
+        </conversion>-->
       </plugin>
     </gazebo>
-    <gazebo reference="${robot_namespace}/thruster_${thruster_id}">
+    <gazebo reference="${namespace}/thruster_${thruster_id}">
       <selfCollide>false</selfCollide>
     </gazebo>
   </xacro:macro>
-</robot>
+</robot>-->

Commit message: Delete the vibrations, changing the solver in gazebo

File: mur_description/urdf/mur_actuators.xacro (robot description, xacro)
@@ -28,14 +28,14 @@
     </xacro:macro>
     <xacro:thruster_macro namespace="${namespace}" thruster_id="0">
-        <origin xyz="0.197 0.18022 0.074" rpy="0 ${-pi/2} 0" />
+        <origin xyz="0.18022 0.197 0.074" rpy="0 ${-pi/2} 0" />
     </xacro:thruster_macro>
     <xacro:thruster_macro namespace="${namespace}" thruster_id="1">
-        <origin xyz="0.197 -0.18022 0.074" rpy="0 ${-pi/2} 0" />
+        <origin xyz="0.18022 -0.197 0.074" rpy="0 ${-pi/2} 0" />
     </xacro:thruster_macro>
     <xacro:thruster_macro namespace="${namespace}" thruster_id="2">
-        <origin xyz="-0.197 -0.18022 0.074" rpy="0 ${-pi/2} 0" />
+        <origin xyz="-0.18022 -0.197 0.074" rpy="0 ${-pi/2} 0" />
     </xacro:thruster_macro>
     <xacro:thruster_macro namespace="${namespace}" thruster_id="3">
-        <origin xyz="-0.197 0.18022 0.074" rpy="0 ${-pi/2} 0" />
+        <origin xyz="-0.18022 0.197 0.074" rpy="0 ${-pi/2} 0" />
     </xacro:thruster_macro>
 </robot>

File: mur_description/urdf/mur_base.xacro (robot description, xacro)
@@ -17,5 +17,5 @@
         <link name="${namespace}/base_link">
             <visual>
-                <origin xyz="0 0 0" rpy="0 0 0"/>
+                <origin xyz="0 0 0" rpy="0 0 -1.57"/>
                 <geometry>
                     <mesh filename="${visual_mesh_file}" scale="1 1 1" />
@@ -23,5 +23,5 @@
             </visual>
             <collision>
-                <origin xyz="0 0 0" rpy="0 0 0"/>
+                <origin xyz="0 0 0" rpy="0 0 -1.57"/>
                     <geometry>
                         <mesh filename="${collision_mesh_file}" scale="1 1 1" />

File: mur_description/urdf/mur_sensors.xacro (robot description, xacro)
@@ -29,5 +29,5 @@
         scale="0.5">
         <inertia ixx="0.00001" ixy="0.0" ixz="0.0" iyy="0.00001" iyz="0.0" izz="0.00001" />
-        <origin xyz="0.05 0.160 0" rpy="0 0 ${pi/2}"/>
+        <origin xyz="0.160 0.05 0" rpy="0 0 0"/>
     </xacro:regular_camera_plugin_macro>
     <!-- Mount a GPS.

Commit message: Recognize the aruco markers

File: mur_description/urdf/mur_actuators.xacro (robot description, xacro)
@@ -28,14 +28,14 @@
     </xacro:macro>
     <xacro:thruster_macro namespace="${namespace}" thruster_id="0">
-        <origin xyz="0.18022 0.197 0.074" rpy="0 ${-pi/2} 0" />
+        <origin xyz="0.197 0.18022 0.074" rpy="0 ${-pi/2} 0" />
     </xacro:thruster_macro>
     <xacro:thruster_macro namespace="${namespace}" thruster_id="1">
-        <origin xyz="0.18022 -0.197 0.074" rpy="0 ${-pi/2} 0" />
+        <origin xyz="-0.197 0.18022 0.074" rpy="0 ${-pi/2} 0" />
     </xacro:thruster_macro>
     <xacro:thruster_macro namespace="${namespace}" thruster_id="2">
-        <origin xyz="-0.18022 -0.197 0.074" rpy="0 ${-pi/2} 0" />
+        <origin xyz="-0.197 -0.18022 0.074" rpy="0 ${-pi/2} 0" />
     </xacro:thruster_macro>
     <xacro:thruster_macro namespace="${namespace}" thruster_id="3">
-        <origin xyz="-0.18022 0.197 0.074" rpy="0 ${-pi/2} 0" />
+        <origin xyz="0.197 -0.18022 0.074" rpy="0 ${-pi/2} 0" />
     </xacro:thruster_macro>
 </robot>

File: mur_description/urdf/mur_base.xacro (robot description, xacro)
@@ -17,5 +17,5 @@
         <link name="${namespace}/base_link">
             <visual>
-                <origin xyz="0 0 0" rpy="0 0 -1.57"/>
+                <origin xyz="0 0 0" rpy="0 0 0"/>
                 <geometry>
                     <mesh filename="${visual_mesh_file}" scale="1 1 1" />
@@ -23,5 +23,5 @@
             </visual>
             <collision>
-                <origin xyz="0 0 0" rpy="0 0 -1.57"/>
+                <origin xyz="0 0 0" rpy="0 0 0"/>
                     <geometry>
                         <mesh filename="${collision_mesh_file}" scale="1 1 1" />

File: mur_description/urdf/mur_sensors.xacro (robot description, xacro)
@@ -21,13 +21,13 @@
         parent_link="${namespace}/base_link"
         topic="camera"
-        mass="0.015"
+        mass="0.1"
         update_rate="30"
-        hfov="1.8125"
+        hfov="1.5125"
         width="768"
         height="492"
         stddev="0.02"
-        scale="0.5">
+        scale="1.0">
         <inertia ixx="0.00001" ixy="0.0" ixz="0.0" iyy="0.00001" iyz="0.0" izz="0.00001" />
-        <origin xyz="0.160 0.05 0" rpy="0 0 0"/>
+        <origin xyz="0.055 0.160 0" rpy="0 0 ${0.5*pi}"/>
     </xacro:regular_camera_plugin_macro>
     <!-- Mount a GPS.

Commit message: Checked stabilization

File: mur_description/urdf/mur_actuators.xacro (robot description, xacro)
@@ -30,7 +30,4 @@
         <origin xyz="0.197 0.18022 0.074" rpy="0 ${-pi/2} 0" />
     </xacro:thruster_macro>
-    <xacro:thruster_macro namespace="${namespace}" thruster_id="3">
-        <origin xyz="-0.197 0.18022 0.074" rpy="0 ${-pi/2} 0" />
-    </xacro:thruster_macro>
     <xacro:thruster_macro namespace="${namespace}" thruster_id="2">
         <origin xyz="-0.197 -0.18022 0.074" rpy="0 ${-pi/2} 0" />
@@ -39,3 +36,6 @@
         <origin xyz="0.197 -0.18022 0.074" rpy="0 ${-pi/2} 0" />
     </xacro:thruster_macro>
+    <xacro:thruster_macro namespace="${namespace}" thruster_id="3">
+        <origin xyz="-0.197 0.18022 0.074" rpy="0 ${-pi/2} 0" />
+    </xacro:thruster_macro>
 </robot>

File: mur_description/urdf/mur_base_ident.xacro (robot description, xacro)
@@ -42,5 +42,5 @@
           <child link="${namespace}/arm_base_link" />
           <origin xyz="0 0 0" rpy="0 0 0"/>
-          <axis xyz="1 0 0"/>
+          <axis xyz="1 1 0"/>
           <limit effort="9999999999999" velocity="999999999999"/>
         </joint>

Commit message: arm was included in simulation

File: mur_description/urdf/mur_actuators.xacro (robot description, xacro)
@@ -8,5 +8,5 @@
           aware that Gazebo does not use the SNAME convention per default.
     -->
-    <xacro:property name="prop_mesh_file" value="file://$(find mur_description)/mesh/mur_prop.dae"/>
+    <xacro:property name="prop_mesh_file" value="file://$(find mur_description)/meshes/mur_prop.dae"/>
     <xacro:macro name="thruster_macro"
       params="namespace thruster_id *origin">

File: mur_description/urdf/mur_actuators_5.xacro (robot description, xacro)
@@ -8,5 +8,5 @@
           aware that Gazebo does not use the SNAME convention per default.
     -->
-    <xacro:property name="prop_mesh_file" value="file://$(find mur_description)/mesh/mur_prop.dae"/>
+    <xacro:property name="prop_mesh_file" value="file://$(find mur_description)/meshes/mur_prop.dae"/>
     <xacro:macro name="thruster_macro"
       params="namespace thruster_id *origin">

File: mur_description/urdf/mur_base.xacro (robot description, xacro)
@@ -11,7 +11,7 @@
     <xacro:property name="cob" value="0 0 0"/>
     <xacro:property name="rho" value="1027.0"/>
-    <xacro:property name="visual_mesh_file" value="file://$(find mur_description)/mesh/mur.dae"/>
-    <xacro:property name="collision_mesh_file" value="file://$(find mur_description)/mesh/mur.dae"/>
-    <xacro:property name="prop_mesh_file" value="file://$(find mur_description)/mesh/mur_prop.dae"/>
+    <xacro:property name="visual_mesh_file" value="file://$(find mur_description)/meshes/mur.dae"/>
+    <xacro:property name="collision_mesh_file" value="file://$(find mur_description)/meshes/mur.dae"/>
+    <xacro:property name="prop_mesh_file" value="file://$(find mur_description)/meshes/mur_prop.dae"/>
     <xacro:macro name="mur_base" params="namespace debug">
         <link name="${namespace}/base_link">

File: mur_description/urdf/mur_base_5.xacro (robot description, xacro)
@@ -11,7 +11,8 @@
     <xacro:property name="cob" value="0 0.005 0.075"/>
     <xacro:property name="rho" value="1000.0"/>
-    <xacro:property name="visual_mesh_file" value="file://$(find mur_description)/mesh/mur_5.dae"/>
-    <xacro:property name="collision_mesh_file" value="file://$(find mur_description)/mesh/mur_5.dae"/>
+    <xacro:property name="visual_mesh_file" value="file://$(find mur_description)/meshes/mur_5.dae"/>
+    <xacro:property name="collision_mesh_file" value="file://$(find mur_description)/meshes/mur_5.dae"/>
     <xacro:macro name="mur_base_5" params="namespace debug">
+        <!-- Base link definition -->
         <link name="${namespace}/base_link">
             <visual>
@@ -33,4 +34,62 @@
                        iyy="0.1496" iyz="0"
                        izz="0.320" />
+            </inertial>
+        </link>
+        <joint name="base_joint" type="revolute">
+            <axis xyz="1 0 0"/>
+            <origin xyz="0 -0.079 -0.1045" rpy="0.92 0 0"/>
+            <parent link="${namespace}/base_link"/>
+            <child link="${namespace}/arm/link"/>
+            <calibration rising="0.0"/>
+            <dynamics damping="1.0" friction="2.0"/>
+            <limit effort="10" velocity="0.025" lower="-6.28" upper="6.28" />
+        </joint>
+        <!-- Link definition -->
+        <link name="${namespace}/arm/link">
+            <visual>
+                <origin xyz="0 0 0" rpy="0 0 0"/>
+                <geometry>
+                  <mesh filename="file://$(find mur_description)/meshes/link.dae" scale="1 1 1" />
+                </geometry>
+            </visual>
+            <collision>
+                <origin xyz="0 0 0" rpy="0 0 0"/>
+                <geometry>
+                  <mesh filename="file://$(find mur_description)/meshes/link.dae" scale="1 1 1" />
+                </geometry>
+            </collision>
+            <inertial>
+              <mass value="0.191" />
+              <origin xyz="0 0 0" rpy="0 0 0"/>
+              <inertia ixx="0.000540" ixy="0" ixz="0.000026"
+                       iyy="0.000554" iyz="0"
+                       izz="0.000035" />
+            </inertial>
+        </link>
+        <joint name="gripper_joint" type="fixed">
+            <origin xyz="0.0175 0 -0.18" rpy="0 0 0"/>
+            <parent link="${namespace}/arm/link"/>
+            <child link="${namespace}/arm/gripper"/>
+        </joint>
+        <!-- Gripper definition -->
+        <link name="${namespace}/arm/gripper">
+            <visual>
+                <origin xyz="0 0 0.005" rpy="0 3.141592 0"/>
+                <geometry>
+                  <mesh filename="file://$(find mur_description)/meshes/gripper.dae" scale="1 1 1" />
+                </geometry>
+            </visual>
+            <collision>
+                <origin xyz="0 0 0.005" rpy="0 3.141592 0"/>
+                <geometry>
+                  <mesh filename="file://$(find mur_description)/meshes/gripper.dae" scale="1 1 1" />
+                </geometry>
+            </collision>
+            <inertial>
+              <mass value="0.185" />
+              <origin xyz="0 0 0" rpy="0 0 0"/>
+              <inertia ixx="0.000299" ixy="0" ixz="0"
+                       iyy="0.000299" iyz="0"
+                       izz="0.000123" />
             </inertial>
         </link>
@@ -72,5 +131,18 @@
           </link>
         </plugin>
+        <plugin name="${namespace}_arm" filename="libgazebo_ros_control.so">
+          <robotNamespace>${namespace}</robotNamespace>
+        </plugin>
       </gazebo>
+      <!-- Transmission -->
+      <transmission name="base_to_link_trans">
+        <type>transmission_interface/SimpleTransmission</type>
+        <actuator name="motor1">
+          <mechanicalReduction>1</mechanicalReduction>
+        </actuator>
+        <joint name="base_joint">
+          <hardwareInterface>EffortJointInterface</hardwareInterface>
+        </joint>
+      </transmission>
       <xacro:include filename="$(find mur_description)/urdf/mur_sensors.xacro"/>
       <xacro:include filename="$(find mur_description)/urdf/mur_actuators_5.xacro"/>

File: mur_description/urdf/mur_base_ident.xacro (robot description, xacro)
@@ -11,7 +11,7 @@
     <xacro:property name="cob" value="0 0 0"/>
     <xacro:property name="rho" value="1027.0"/>
-    <xacro:property name="visual_mesh_file" value="file://$(find mur_description)/mesh/mur_5.dae"/>
-    <xacro:property name="collision_mesh_file" value="file://$(find mur_description)/mesh/mur_5.dae"/>
-    <xacro:property name="prop_mesh_file" value="file://$(find mur_description)/mesh/mur_prop.dae"/>
+    <xacro:property name="visual_mesh_file" value="file://$(find mur_description)/meshes/mur_5.dae"/>
+    <xacro:property name="collision_mesh_file" value="file://$(find mur_description)/meshes/mur_5.dae"/>
+    <xacro:property name="prop_mesh_file" value="file://$(find mur_description)/meshes/mur_prop.dae"/>
     <xacro:macro name="mur_base_ident" params="namespace debug">
     <!-- THE ROBOT -->

File: mur_description/urdf/mur_sensors.xacro (robot description, xacro)
@@ -23,5 +23,5 @@
         <visual>
           <geometry>
-            <mesh filename="file://$(find mur_description)/mesh/Micron DST Sonar.dae" scale="1 1 1"/>
+            <mesh filename="file://$(find mur_description)/meshes/Micron DST Sonar.dae" scale="1 1 1"/>
           </geometry>
         </visual>

File: mur_description/urdf/mur_snippets.xacro (robot description, xacro)
@@ -7,5 +7,5 @@
   over propeller's frame X-axis in DAE (Collada) or STL format.
   -->
-  <xacro:property name="prop_mesh_file" value="file://$(find mur_description)/mesh/mur_prop.dae"/>
+  <xacro:property name="prop_mesh_file" value="file://$(find mur_description)/meshes/mur_prop.dae"/>
   <!--
     Thruster macro with integration of joint and link. The thrusters should
@@ -150,3 +150,3 @@
     </gazebo>
   </xacro:macro>
-</robot>-->
+</robot>
